File: src/hw/board_files/KuhnYork_rev_0_1/pocket-caddy.kicad_sch (KiCad schematic)
At the start: 6 parts

Commit message: rev0.1 done
Parts:
- removed TP3: SD_CS_TP, TestPoint:TestPoint_Pad_D1.5mm, symbol Connector:TestPoint
- removed TP4: SPI_MOSI_TP, TestPoint:TestPoint_Pad_D1.5mm, symbol Connector:TestPoint
- removed TP5: SPI_MISO_TP, TestPoint:TestPoint_Pad_D1.5mm, symbol Connector:TestPoint
- removed TP6: SPI_SCK_TP, TestPoint:TestPoint_Pad_D1.5mm, symbol Connector:TestPoint
- TP1, TP2: footprint TestPoint:TestPoint_Pad_D1.5mm -> TestPoint:TestPoint_Pad_D1.0mm
Other:
- sheet Microcontroller ports: added none; removed ESP32_RX, ESP32_TX
- sheet Peripherals ports: added NTC_THERM; removed none
- sheet USB-C and Power ports: added NTC_THERM; removed ESP32_RX, ESP32_TX
