File: src/hw/board_files/KuhnYork_rev_0_1/power.kicad_sch (KiCad schematic)
At the start: 33 parts, among them J1 USB_C_Receptacle_USB2.0_14P, J2 Screw_Terminal_01x03, J3 Conn_01x03_Pin, SW1 SW_PWR, U1 MCP73871, U2 TPS63031DSKR

Commit message: rev0.1 done
Parts:
- removed BT1: LiPo, Connector_JST:JST_PH_S2B-PH-K_1x02_P2.00mm_Horizontal, symbol Device:Battery_Cell
- removed J2: Screw_Terminal_01x03, TerminalBlock_Phoenix:TerminalBlock_Phoenix_MPT-0,5-3-2.54_1x03_P2.54mm_Horizontal, symbol Connector:Screw_Terminal_01x03
- removed J3: Conn_01x03_Pin, Connector_PinHeader_2.54mm:PinHeader_1x03_P2.54mm_Vertical, symbol Connector:Conn_01x03_Pin
- TP3: renamed from TP7; footprint TestPoint:TestPoint_Pad_D1.5mm -> TestPoint:TestPoint_Pad_D1.0mm
- renumbered R3 to R2, R2 to R3, R6 to R5, R7 to R6, R5 to R7
Connections:
- net V_SYS: now also F1.1
Other:
- note removed: "LiPo Battery"
- moved on the sheet: C4, C5, C6, C7, D2, D5, F1, J1, L1, NT1, R1, R10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
